File: kicad/a2000Serotina.kicad_pcb (KiCad board)
At the start: 2 copper layers, 232 parts, among them J1 KCDX-5S-S2, U1 Teensy++2.0_(C)

Commit message: All switches now placed.
Parts:
- MX58: footprint MX_Alps_Hybrid:MX-1U-NoLED -> MX_Alps_Hybrid:MX-2U-NoLED
- moved MX97 813.6 mm to (816.0, 76.2), turned to 90 degrees
- moved MX103 759.1 mm to (816.0, 38.1), turned to 270 degrees
- moved D97 735.3 mm to (819.9, 95.2), turned to 180 degrees
- moved MX85 731.8 mm to (777.9, 28.6)
- moved MX95 712.1 mm to (796.9, 28.6)
- moved MX89 709.8 mm to (796.9, 66.7)
- moved MX76 706.6 mm to (777.9, 47.6)
- moved D95 705.2 mm to (793.0, 38.1)
- moved MX58 695.4 mm to (768.4, 85.7)
- moved D103 678.5 mm to (812.8, 57.1)
- moved MX66 674.8 mm to (758.8, 47.6)
- moved MX12 674.1 mm to (670.7, 85.7)
- moved MX78 672.7 mm to (777.9, 66.7)
- moved D89 667.4 mm to (793.0, 76.2)
- moved MX87 651.5 mm to (796.9, 47.6)
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
Commit message: All Components now placed on PCB
Parts:
- moved R11 838.6 mm to (808.0, -5.56)
- moved R8 699.0 mm to (729.5, 49.2)
- moved R4 698.7 mm to (702.5, 49.2), turned to 180 degrees
- moved R9 684.6 mm to (729.6, 54.0)
- moved R10 684.4 mm to (729.5, 58.7)
- moved R5 684.2 mm to (702.5, 54.0), turned to 180 degrees
- moved R6 684.1 mm to (702.5, 58.7), turned to 180 degrees
- moved R7 669.6 mm to (702.5, 63.5), turned to 180 degrees
- moved LED8 641.5 mm to (823.1, -5.56), turned to 180 degrees
- moved R3 603.3 mm to (611.2, 81.0), turned to 270 degrees
- moved LED7 505.5 mm to (744.5, 58.7), turned to 180 degrees
- moved LED2 460.8 mm to (687.4, 54.0)
- moved R12 456.0 mm to (430.2, 53.2), turned to 90 degrees
- moved R2 452.2 mm to (444.5, 81.0), turned to 270 degrees
- moved LED5 444.6 mm to (744.5, 49.2), turned to 180 degrees
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
Commit message: Auto routing complete
Parts:
- moved MX28 2.38 mm to (670.7, 38.1)
- moved D28 1.59 mm to (666.8, 57.1)
- moved U1 1.12 mm to (800.1, -19.8)
- moved J1 0.79 mm to (766.8, -15.1)
- moved R11 0.79 mm to (808.8, -5.56)
- moved LED8 0.79 mm to (823.9, -5.56)
Routing:
- net COL0: track 0.00 -> 745.7 mm
- net COL2: track 0.00 -> 686.1 mm, vias 0 -> 1
- net COL4: track 0.00 -> 683.4 mm, vias 0 -> 1
- net COL5: track 0.00 -> 671.8 mm, vias 0 -> 2
- net COL3: track 0.00 -> 664.4 mm, vias 0 -> 2
- net COL1: track 0.00 -> 629.7 mm
- net GND: track 0.00 -> 586.2 mm
- net COL8: track 0.00 -> 489.2 mm, vias 0 -> 1
- net COL7: track 0.00 -> 487.3 mm, vias 0 -> 2
- net COL6: track 0.00 -> 484.1 mm, vias 0 -> 2
- net ROW8: track 0.00 -> 481.9 mm, vias 0 -> 1
- net ROW10: track 0.00 -> 467.9 mm
- net LALT: track 0.00 -> 466.7 mm, vias 0 -> 1
- net ROW6: track 0.00 -> 456.7 mm, vias 0 -> 1
- net ROW2: track 0.00 -> 449.9 mm
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Other:
- board outline added: 436.6 x 131.8 mm
- net class Default: trace_width 0.25 -> 0.254
- net class Power added: clearance 0.2, trace_width 0.381, via_dia 0.8, via_drill 0.4
- board text added: "A2000 Serotina V1.0 - created by grshaw and bperryman with thanks to Rob Taylor and LIV2"

Commit message: Fix PCB layout
Move Diodes that are too close to Stabilizer drill holes.
Parts:
- moved D28 27.7 mm to (654.0, 32.5), turned to 90 degrees
- moved D10 14.3 mm to (592.1, 70.6), turned to 90 degrees
- moved D97 7.94 mm to (812.0, 95.2), turned to 0 degrees
- turned MX103 to 90 degrees
- turned MX28 to 90 degrees
Routing:
- net COL0: track 745.7 -> 0.00 mm
- net COL2: track 686.1 -> 0.00 mm, vias 1 -> 0
- net COL4: track 683.4 -> 0.00 mm, vias 1 -> 0
- net COL5: track 671.8 -> 0.00 mm, vias 2 -> 0
- net COL3: track 664.4 -> 0.00 mm, vias 2 -> 0
- net COL1: track 629.7 -> 0.00 mm
- net GND: track 586.2 -> 0.00 mm
- net COL8: track 489.2 -> 0.00 mm, vias 1 -> 0
- net COL7: track 487.3 -> 0.00 mm, vias 2 -> 0
- net COL6: track 484.1 -> 0.00 mm, vias 2 -> 0
- net ROW8: track 481.9 -> 0.00 mm, vias 1 -> 0
- net ROW10: track 467.9 -> 0.00 mm
- net LALT: track 466.7 -> 0.00 mm, vias 1 -> 0
- net ROW6: track 456.7 -> 0.00 mm, vias 1 -> 0
- net ROW2: track 449.9 -> 0.00 mm
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
Commit message: Generated Gerber Files and Bill of Materials
Routing:
- net COL0: track 0.00 -> 728.0 mm
- net COL2: track 0.00 -> 715.9 mm, vias 0 -> 1
- net COL4: track 0.00 -> 689.0 mm, vias 0 -> 1
- net COL3: track 0.00 -> 684.3 mm, vias 0 -> 1
- net COL5: track 0.00 -> 649.9 mm, vias 0 -> 1
- net COL1: track 0.00 -> 634.2 mm
- net GND: track 0.00 -> 586.7 mm
- net COL7: track 0.00 -> 503.7 mm, vias 0 -> 1
- net COL6: track 0.00 -> 492.1 mm, vias 0 -> 1
- net COL8: track 0.00 -> 490.3 mm, vias 0 -> 1
- net ROW8: track 0.00 -> 470.8 mm, vias 0 -> 1
- net ROW10: track 0.00 -> 469.6 mm
- net ROW2: track 0.00 -> 450.7 mm
- net ROW6: track 0.00 -> 449.5 mm, vias 0 -> 1
- net ROW4: track 0.00 -> 445.0 mm, vias 0 -> 1
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
Commit message: Added Text Labels to Front Silkscreen
Added letter labels for Mx Switches
Added labels for LEDs
Sorted out Resistor footprints so that vaules are visible on Front Silkscreen.
Other:
- board size 436.6 x 131.8 mm -> 439.7 x 134.9 mm
- board text added: "0"
- board text added: "1"
- board text added: "2"
- board text added: "3"
- board text added: "4"
- board text added: "5"
- board text added: "6"
- board text added: "7"
- board text added: "8"
- board text added: "9"
- board text added: "A"
- board text added: "B"
- board text added: "BSLS \"
- board text added: "BSPC"
- board text added: "C"
- board text added: "CAPS"
- board text added: "COMM ,"
- board text added: "D"
- board text added: "DEL / BLANK"
- board text added: "DOT ."
- board text added: "DOWN"
- board text added: "E"
- board text added: "END / BLANK"
- board text added: "ENT"
- board text added: "EQL ="
- board text added: "ESC"
- board text added: "Esc"
- board text added: "F"
- board text added: "F1"
- board text added: "F10"
- board text added: "F11 / BLANK"
- board text added: "F12 / BLANK"
- board text added: "F2"
- board text added: "F3"
- board text added: "F4"
- board text added: "F5"
- board text added: "F6"
- board text added: "F7"
- board text added: "F8"
- board text added: "F9"
- board text added: "G"
- board text added: "GRV `"
- board text added: "H"
- board text added: "HOME / DEL"
- board text added: "I"
- board text added: "INS / DEL"
- board text added: "J"
- board text added: "K"
- board text added: "KCLK"
- board text added: "KDAT"
- board text added: "L"
- board text added: "LALT / LAMI"
- board text added: "LBRC ["
- board text added: "LCTRL"
- board text added: "LEFT"
- board text added: "LGUI / LALT"
- board text added: "LSHFT"
- board text added: "M"
- board text added: "MENU / RALT"
- board text added: "MIN -"
- board text added: "N"
- board text added: "NLCK"
- board text added: "NLCK / BLANK"
- board text added: "NUHS / BLANK"
- board text added: "O"
- board text added: "P"
- board text added: "PAST *"
- board text added: "PAUS / BLANK"
- board text added: "PDOT"
- board text added: "PENT"
- board text added: "PGDN / BLANK"
- board text added: "PGUP / HELP"
- board text added: "PMNS -"
- board text added: "POWER"
- board text added: "PPLS +"
- board text added: "PSCR / BLANK"
- board text added: "PSLS /"
- board text added: "Q"
- board text added: "QUOT / AT"
- board text added: "R"
- board text added: "RALT / BLANK"
- board text added: "RBRC ]"
- board text added: "RCTRL"
- board text added: "RGHT"
- board text added: "RGUI / RAMI"
- board text added: "RSHIFT"
- board text added: "S"
- board text added: "SCLN ;"
- board text added: "SLCK"
- board text added: "SLCK / BLANK"
- board text added: "SLSH /"
- board text added: "SPC"
- board text added: "STA1"
- board text added: "STA2"
- board text added: "STA3"
- board text added: "T"
- board text added: "TAB"
- board text added: "U"
- board text added: "UP"
- board text added: "V"
- board text added: "W"
- board text added: "X"
- board text added: "Y"
- board text added: "Z"

Commit message: Update to PCB
Moved DIN socket and CPU nearer to edge of PCB.
Parts:
- moved J1 5.56 mm to (766.8, -20.6)
- moved LED8 3.97 mm to (827.9, -5.56)
- moved R11 3.97 mm to (812.8, -5.56)
- moved U1 3.97 mm to (804.1, -19.8)
Routing:
- net ROW5: track 321.2 -> 284.5 mm
- net LCTRL: track 433.1 -> 468.3 mm, vias 1 -> 0
- net COL8: track 490.3 -> 516.3 mm, vias 1 -> 0
- net STA1: track 124.3 -> 146.3 mm
- net COL2: track 715.9 -> 696.5 mm, vias 1 -> 2
- net VCC: track 65.6 -> 84.4 mm
- net LALT: track 424.6 -> 405.9 mm
- net KDAT: track 107.1 -> 124.7 mm
- net RGUI: track 276.2 -> 290.0 mm
- net COL3: track 684.3 -> 671.7 mm
- net GND: track 586.7 -> 598.9 mm
- net KCLK: track 107.3 -> 119.1 mm
- net ROW4: track 445.0 -> 455.4 mm
- net ROW8: track 470.8 -> 460.5 mm
- net SCLCK: track 116.1 -> 124.1 mm
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
Commit message: Change Row 6 Pin from D6 to F2
D6 lights the LED on the Teensy 2.0 ++ - better to have D6 control a LED.
Connections:
- U1 pad 29: SCLCK -> ROW6
- U1 pad 9: ROW6 -> SCLCK
Routing:
- net COL2: track 696.5 -> 729.5 mm, vias 2 -> 1
- net ROW6: track 446.1 -> 425.0 mm
- net SCLCK: track 124.1 -> 144.4 mm, vias 0 -> 1
- net ROW9: track 375.9 -> 357.8 mm
- net ROW5: track 284.5 -> 301.3 mm
- net COL4: track 689.6 -> 674.0 mm, vias 0 -> 1
- net COL9: track 401.1 -> 416.6 mm
- net ROW11: track 275.3 -> 262.6 mm
- net GND: track 598.9 -> 588.3 mm
- net COL6: track 489.1 -> 499.0 mm
- net ROW10: track 467.6 -> 476.7 mm
- net COL10: track 265.4 -> 273.7 mm
- net COL0: track 729.1 -> 736.2 mm
- net ROW7: track 334.1 -> 327.2 mm, vias 0 -> 1
- net VCC: track 84.4 -> 77.5 mm
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