File: kicad/a2000Serotina.kicad_pcb (KiCad board)
At the start: 2 copper layers, 439.7 x 134.9 mm, 232 parts, among them J1 KCDX-5S-S2, U1 Teensy++2.0_(C)

Commit message: Updated column / row layout of switches
Now much more regular on the bottom rows.
Connections:
- D10 pad 1: ROW9 -> ROW8
- D18 pad 1: ROW7 -> ROW6
- D2 pad 1: ROW1 -> ROW0
- D20 pad 1: ROW9 -> ROW8
- D24 pad 1: ROW1 -> ROW0
- D30 pad 1: ROW7 -> ROW6
- D69 pad 1: ROW10 -> ROW11
- D79 pad 1: ROW10 -> ROW11
- D8 pad 1: ROW7 -> ROW6
- MX10 pad 1: COL0 -> COL9
- MX12 pad 1: COL0 -> COL2
- MX18 pad 1: COL1 -> COL9
- MX2 pad 1: COL0 -> COL9
- MX20 pad 1: COL1 -> COL10
- MX22 pad 1: COL1 -> COL3
- MX24 pad 1: COL2 -> COL10
- MX30 pad 1: COL2 -> COL10
- MX32 pad 1: COL2 -> COL0
- MX34 pad 1: COL2 -> COL4
- MX36 pad 1: COL3 -> COL0
- MX42 pad 1: COL3 -> COL0
- MX44 pad 1: COL3 -> COL1
- MX45 pad 1: COL3 -> COL6
- MX46 pad 1: COL3 -> COL5
- MX48 pad 1: COL4 -> COL1
- MX54 pad 1: COL4 -> COL1
- MX57 pad 1: COL4 -> COL10
- MX58 pad 1: COL4 -> COL6
- MX60 pad 1: COL5 -> COL2
- MX66 pad 1: COL5 -> COL6
- MX68 pad 1: COL5 -> COL6
- MX69 pad 1: COL5 -> COL0
- MX70 pad 1: COL5 -> COL8
- MX76 pad 1: COL6 -> COL7
- MX78 pad 1: COL6 -> COL7
- MX79 pad 1: COL6 -> COL1
- MX8 pad 1: COL0 -> COL8
- MX80 pad 1: COL7 -> COL6
- MX81 pad 1: COL7 -> COL3
- MX87 pad 1: COL7 -> COL8
- MX89 pad 1: COL7 -> COL8
- MX90 pad 1: COL8 -> COL7
- MX91 pad 1: COL8 -> COL4
- MX97 pad 1: COL8 -> COL9
- MX98 pad 1: COL9 -> COL8
- MX99 pad 1: COL9 -> COL5
- U1 pad 10: ROW7 -> CPLCK
- U1 pad 13: ROW8 -> COL3
- U1 pad 14: ROW9 -> COL4
- U1 pad 15: ROW10 -> COL5
- U1 pad 16: ROW11 -> COL6
- U1 pad 17: COL0 -> COL7
- U1 pad 18: COL1 -> COL8
- U1 pad 19: COL2 -> COL9
- U1 pad 20: COL3 -> COL10
- U1 pad 29: ROW6 -> COL2
- U1 pad 3: ROW0 -> ROW3
- U1 pad 30: CPLCK -> COL1
- U1 pad 31: NMLCK -> COL0
- U1 pad 36: COL4 -> ROW0
- U1 pad 37: COL5 -> ROW1
- U1 pad 38: COL6 -> ROW2
- U1 pad 39: COL7 -> ROW4
- U1 pad 4: ROW1 -> ROW5
- U1 pad 40: COL8 -> ROW6
- U1 pad 41: COL9 -> ROW8
- U1 pad 42: COL10 -> ROW10
- U1 pad 5: ROW2 -> ROW7
- U1 pad 6: ROW3 -> ROW9
- U1 pad 7: ROW4 -> ROW11
- U1 pad 8: ROW5 -> NMLCK
Routing:
- net COL4: track 674.0 -> 538.5 mm, vias 1 -> 0
- net COL5: track 644.5 -> 511.8 mm, vias 1 -> 0
- net COL2: track 729.5 -> 597.4 mm
- net COL3: track 674.1 -> 554.4 mm
- net COL0: track 736.2 -> 638.9 mm
- net ROW1: track 251.1 -> 188.6 mm
- net ROW7: track 327.2 -> 269.7 mm, vias 1 -> 0
- net COL7: track 504.6 -> 447.6 mm, vias 1 -> 0
- net NMLCK: track 139.0 -> 195.1 mm, vias 1 -> 0
- net COL9: track 416.6 -> 471.0 mm
- net COL8: track 516.9 -> 463.7 mm
- net ROW11: track 262.6 -> 312.2 mm
- net ROW6: track 425.0 -> 464.5 mm, vias 1 -> 0
- net COL1: track 633.4 -> 601.2 mm
- net COL10: track 273.7 -> 301.5 mm
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
Commit message: Add Mounting holes
Parts:
- added H1: MountingHole, MountingHole:MountingHole_2.2mm_M2, F.Cu at (492.1, -3.17)
- added H2: MountingHole, MountingHole:MountingHole_2.2mm_M2, F.Cu at (458.8, 57.1)
- added H3: MountingHole, MountingHole:MountingHole_2.2mm_M2, F.Cu at (554.0, 57.1)
- added H4: MountingHole, MountingHole:MountingHole_2.2mm_M2, F.Cu at (768.4, 57.1)
- added H5: MountingHole, MountingHole:MountingHole_5.3mm_M5, F.Cu at (413.5, -3.17)
- added H6: MountingHole, MountingHole:MountingHole_5.3mm_M5, F.Cu at (584.2, -3.17)
- added H7: MountingHole, MountingHole:MountingHole_5.3mm_M5, F.Cu at (808.0, -3.17)
- moved D45 57.2 mm to (523.9, 76.2), turned to 0 degrees
- moved D97 38.1 mm to (812.8, 57.1)
- moved D103 38.1 mm to (812.0, 19.1)
- moved LED8 38.1 mm to (789.8, -5.56)
- moved R11 38.1 mm to (774.7, -5.56)
- moved D58 26.5 mm to (764.4, 76.2), turned to 0 degrees
- moved D44 23.1 mm to (652.5, 57.1), turned to 0 degrees
- moved D33 20.3 mm to (452.4, 76.2), turned to 0 degrees
- moved D26 20.2 mm to (659.6, 0.00), turned to 0 degrees
- moved D100 19.6 mm to (569.1, 0.00)
- moved D101 19.5 mm to (816.0, 0.00)
- moved D3 19.5 mm to (398.5, 0.00)
- moved D10 19.1 mm to (578.6, 57.1), turned to 0 degrees
- moved D68 19.1 mm to (754.9, 57.1), turned to 0 degrees
- moved D78 19.1 mm to (773.9, 57.1), turned to 0 degrees
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Routing:
- net COL0: track 638.9 -> 0.00 mm
- net COL1: track 601.2 -> 0.00 mm
- net GND: track 599.3 -> 0.00 mm
- net COL2: track 597.4 -> 0.00 mm, vias 1 -> 0
- net COL3: track 554.4 -> 0.00 mm
- net COL4: track 538.5 -> 0.00 mm
- net COL5: track 511.8 -> 0.00 mm
- net ROW10: track 501.7 -> 0.00 mm
- net COL6: track 500.9 -> 0.00 mm
- net ROW8: track 483.5 -> 0.00 mm
- net COL9: track 471.0 -> 0.00 mm
- net ROW6: track 464.5 -> 0.00 mm
- net COL8: track 463.7 -> 0.00 mm
- net LCTRL: track 448.5 -> 0.00 mm, vias 1 -> 0
- net ROW4: track 448.4 -> 0.00 mm
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Other:
- board size 439.7 x 134.9 mm -> 430.2 x 125.4 mm

Commit message: Change 5 Pin Din to right angle pin headers
So that a case will fit on.
Parts:
- H1, H2, H3, H4: footprint MountingHole:MountingHole_2.2mm_M2 -> MountingHole:MountingHole_3.2mm_M3
- H5, H6, H7: footprint MountingHole:MountingHole_5.3mm_M5 -> MountingHole:MountingHole_6.4mm_M6
- J1: value KCDX-5S-S2 -> 90121-0766; footprint SamacSys_Parts:KCDX5SS2 -> SamacSys_Parts:901210766; moved to B.Cu
- U1: moved to B.Cu
- moved R1 281.5 mm to (701.7, 63.5), turned to 180 degrees
- moved R2 257.6 mm to (701.7, 66.7), turned to 180 degrees
- moved R3 91.2 mm to (701.7, 69.8), turned to 180 degrees
- moved D3 20.2 mm to (413.5, 13.5), turned to 90 degrees
- moved D101 16.5 mm to (806.5, 13.5), turned to 90 degrees
- moved D1 16.1 mm to (415.9, -15.1), turned to 90 degrees
- moved D93 14.6 mm to (787.4, 13.5), turned to 90 degrees
- moved J1 11.1 mm to (755.6, -15.9), turned to 270 degrees
- moved D2 10.3 mm to (596.9, -15.1), turned to 90 degrees
- moved D100 5.61 mm to (568.3, 5.56), turned to 270 degrees
- moved R4 4.83 mm to (701.7, 44.4)
- moved R6 4.83 mm to (701.7, 54.0)
- moved R5 4.83 mm to (701.7, 49.2)
- moved R7 4.83 mm to (701.7, 58.7)
- moved LED1 4.83 mm to (686.6, 44.4)
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Connections:
- J1 pad 1: Net-(J1-Pad1) -> GND
- J1 pad 2: KDAT -> VCC
- J1 pad 3: KCLK -> Net-(J1-Pad3)
- J1 pad 4: VCC -> Net-(J1-Pad4)
- J1 pad 5: GND -> KCLK
Routing:
- net COL0: track 0.00 -> 646.3 mm
- net COL2: track 0.00 -> 615.9 mm
- net COL1: track 0.00 -> 600.1 mm
- net COL4: track 0.00 -> 570.5 mm
- net COL3: track 0.00 -> 558.5 mm
- net GND: track 0.00 -> 544.5 mm
- net COL5: track 0.00 -> 530.9 mm
- net COL6: track 0.00 -> 519.4 mm, vias 0 -> 1
- net COL8: track 0.00 -> 467.4 mm
- net COL7: track 0.00 -> 459.7 mm, vias 0 -> 1
- net COL9: track 0.00 -> 459.6 mm
- net ROW10: track 0.00 -> 450.4 mm, vias 0 -> 1
- net ROW8: track 0.00 -> 434.7 mm, vias 0 -> 1
- net CPLCK: track 0.00 -> 415.9 mm, vias 0 -> 1
- net ROW6: track 0.00 -> 410.4 mm, vias 0 -> 1
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Other:
- board text added: "A2000 Serotina V1.1 - created by grshaw and bperryman"
- board text added: "with thanks to LIV2 and Rob Taylor"
- board text removed: "A2000 Serotina V1.0 - created by grshaw and bperryman with thanks to Rob Taylor and LIV2"

Commit message: Move and rotate right angle pin header
Parts:
- moved J1 7.86 mm to (761.2, -10.3), turned to 0 degrees
Routing:
- net COL7: track 459.7 -> 491.2 mm, vias 1 -> 0
- net COL6: track 519.4 -> 550.1 mm
- net COL8: track 467.4 -> 497.3 mm
- net STA2: track 176.4 -> 152.1 mm, vias 0 -> 1
- net COL4: track 570.5 -> 548.4 mm
- net STA3: track 176.3 -> 159.4 mm, vias 0 -> 1
- net RGUI: track 154.3 -> 139.5 mm
- net COL5: track 530.9 -> 517.1 mm, vias 0 -> 1
- net ROW5: track 274.2 -> 260.4 mm
- net ROW10: track 450.4 -> 437.5 mm
- net LCTRL: track 172.0 -> 184.4 mm
- net COL3: track 558.5 -> 567.4 mm
- net ROW3: track 240.5 -> 249.1 mm
- net ROW6: track 410.4 -> 418.6 mm
- net GND: track 544.5 -> 536.7 mm
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Other:
- board text added: "Snip"

Commit message: Updated PCB design, fitting into case
1) Add extra CTRL_LED in Right Ctrl Key  DONE

2) Add extra CAPS_LED in top right  LED6 R9 ( Previously KCLK )  DONE
CAPS_LOCK   NUM_LOCK    SCR_LOCK

3) Move NMLCK + SCLCK LEDs to top right  DONE

4) Fix font on second half of Thank you message  DONE
with thanks to LIV2 and Rob Taylor

5) Update Amiga keys on silkscreen  DONE

6) Move R12 to be in line with all other resistors  DONE

7) Need to move D72 so that it doesn't contact J1   DONE

8) Update Snip Silk screen  DONE

9) Move D3 - too close to MX Switch   DONE

10) Update firmware - add flash of all LEDs for 1.0s on start up...  DONE

12) Remove power LED   DONE

13) Remove KDAT + KCLK LEDS DONE

14) Move big Mounting holes H5, H6 + H7 right 1 square and up 1 square  DONE

15) Move H1 Up by 1mm  DONE

16) Move top row down. Should it be by 1 or 2 squares?  Try just one square   DONE

17) Make PCB wider so that it sits on the shelf properly

18) R10 + R11 missing   DONE
R12 -> R10
R13 -> R11
Parts:
- removed LED7, LED8: LED, LED_THT:LED_D3.0mm
- removed R12: 150, Resistor_THT:R_Axial_DIN0207_L6.3mm_D2.5mm_P10.16mm_Horizontal
- MX12: value MX-NoLED -> MX-LED; footprint MX_Alps_Hybrid:MX-1.25U-NoLED -> MX_Alps_Hybrid:MX-1.25U
- moved LED4 127.6 mm to (797.7, -3.97)
- moved R7 106.6 mm to (790.6, 0.00), turned to 0 degrees
- moved R8 100.4 mm to (825.5, 15.1), turned to 90 degrees
- moved R11 93.6 mm to (702.5, 54.0), turned to 180 degrees
- moved LED5 87.6 mm to (817.6, -3.97), turned to 0 degrees
- moved R9 65.7 mm to (773.1, 0.00)
- moved LED6 63.1 mm to (778.5, -3.97), turned to 0 degrees
- moved LED3 57.4 mm to (743.0, 42.9), turned to 270 degrees
- moved LED2 51.2 mm to (737.4, 42.9), turned to 270 degrees
- moved LED1 44.5 mm to (731.0, 42.9), turned to 270 degrees
- moved R6 41.5 mm to (743.0, 57.9), turned to 90 degrees
- moved R5 36.8 mm to (737.4, 57.9), turned to 90 degrees
- moved R4 32.3 mm to (731.0, 57.9), turned to 90 degrees
- moved R10 27.2 mm to (702.5, 50.8), turned to 180 degrees
- moved R1 22.2 mm to (702.5, 41.3)
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Connections:
- R1 pad 1: LCTRL -> CTRL
- R10 pad 1: KDAT -> CPLCK
- R10 pad 2: Net-(LED7-Pad2) -> Net-(MX7-Pad3)
- R11 pad 1: VCC -> CTRL
- R11 pad 2: Net-(LED8-Pad2) -> Net-(MX12-Pad3)
- R9 pad 1: KCLK -> CPLCK
- U1 pad 11: LCTRL -> CTRL
Routing:
- net CPLCK: track 418.7 -> 134.3 mm, vias 0 -> 1
- net Net-(MX7-Pad3): track 19.5 -> 281.9 mm
- net LCTRL: track 184.4 -> 0.00 mm
- net CTRL: track 0.00 -> 151.4 mm, vias 0 -> 1
- net NMLCK: track 170.8 -> 27.2 mm, vias 0 -> 1
- net KDAT: track 140.2 -> 59.9 mm, vias 1 -> 0
- net KCLK: track 137.3 -> 59.6 mm
- net LALT: track 218.5 -> 143.7 mm
- net Net-(MX12-Pad3): track 0.00 -> 46.3 mm
- net SCLCK: track 114.3 -> 70.4 mm, vias 1 -> 0
- net COL6: track 550.1 -> 522.7 mm
- net COL8: track 497.3 -> 469.9 mm
- net RGUI: track 139.5 -> 112.3 mm
- net GND: track 536.7 -> 563.0 mm, vias 0 -> 1
- net STA2: track 152.1 -> 125.9 mm
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Other:
- board size 430.2 x 125.4 mm -> 434.2 x 131 mm
- board text added: "A2000 Serotina V1.2 - created by grshaw and bperryman"
- board text added: "BSLS"
- board text added: "COMM"
- board text added: "CPLCK"
- board text added: "DEL"
- board text added: "DOT"
- board text added: "END / PLPN"
- board text added: "LBRC"
- board text added: "NMLCK"
- board text added: "NUHS"
- board text added: "PAST"
- board text added: "PGDN / PRPN"
- board text added: "PMNS"
- board text added: "PSLS"
- board text added: "QUOT"
- board text added: "RALT / SPC"
- board text added: "RBRC"
- board text added: "SCLCK"
- board text added: "SCLN"
- board text added: "SLSH"
- board text removed: "A2000 Serotina V1.1 - created by grshaw and bperryman"
- board text removed: "BSLS \"
- board text removed: "COMM ,"
- board text removed: "DEL / BLANK"
- board text removed: "END / BLANK"
- board text removed: "KCLK"
- board text removed: "KDAT"
- board text removed: "LBRC ["
- board text removed: "NLCK"
- board text removed: "NUHS / BLANK"
- board text removed: "PAST *"
- board text removed: "PGDN / BLANK"
- board text removed: "PMNS -"
- board text removed: "POWER"
- board text removed: "PSLS /"
- board text removed: "QUOT / AT"
- board text removed: "RALT / BLANK"
- board text removed: "RBRC ]"
- board text removed: "SCLN ;"
- board text removed: "SLCK"
- board text removed: "SLSH /"

Commit message: V1.3 Design Complete
Parts:
- moved J1 15.4 mm to (758.0, -25.4)
- moved D72 7.94 mm to (754.9, 19.1), turned to 0 degrees
- moved LED4 3.18 mm to (797.7, -7.14)
- moved LED5 3.18 mm to (817.6, -7.14)
- moved LED6 3.18 mm to (778.5, -7.14)
- moved U1 2.38 mm to (799.3, -20.6)
- moved H6 0.79 mm to (585.8, -3.97)
Routing:
- net ROW10: track 430.4 -> 467.1 mm
- net STA3: track 159.6 -> 127.4 mm
- net COL6: track 522.7 -> 553.4 mm, vias 1 -> 0
- net CTRL: track 151.4 -> 171.4 mm
- net ROW6: track 402.8 -> 422.4 mm, vias 0 -> 1
- net RGUI: track 112.3 -> 129.1 mm, vias 0 -> 1
- net ROW9: track 313.2 -> 299.8 mm
- net LALT: track 143.7 -> 155.8 mm
- net ROW8: track 422.1 -> 430.7 mm
- net CPLCK: track 134.3 -> 142.9 mm, vias 1 -> 2
- net VCC: track 18.7 -> 26.7 mm
- net COL4: track 550.0 -> 557.6 mm
- net ROW11: track 314.5 -> 307.3 mm
- net Net-(MX69-Pad3): track 97.7 -> 90.6 mm
- net ROW5: track 286.0 -> 279.5 mm
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Other:
- board size 434.2 x 131 mm -> 434.2 x 131.8 mm
- board text added: "A2000 Serotina V1.3 - created by grshaw and bperryman"
- board text added: "EQL"
- board text added: "MIN"
- board text removed: "A2000 Serotina V1.2 - created by grshaw and bperryman"
- board text removed: "DOT ."
- board text removed: "EQL ="
- board text removed: "MIN -"

Commit message: Change for V1.4
Now uses a mounting plate from WASD.
1) Adjust dimensions to match WASD PCB
2) Make mounting holes bigger so that PCB sits lower
3) Move resistors so that they are not under plate
4) Move Caps Lock LED to rightmost and move Teensy back to top.
5) J1 moved between Enter + Del
6) Stabilizer holes deleted. Costar Stabilizers now attached to Plate.
7) Minimize hole courtyards to pass Design Rules Check
Parts:
- removed LED4, LED5: LED, LED_THT:LED_D3.0mm
- removed R7, R8: 150, Resistor_THT:R_Axial_DIN0207_L6.3mm_D2.5mm_P10.16mm_Horizontal
- H1, H2, H3, H4: footprint MountingHole:MountingHole_3.2mm_M3 -> MountingHole:MountingHole_6.4mm_M6
- H5, H6, H7: footprint MountingHole:MountingHole_6.4mm_M6 -> MountingHole:MountingHole_8.4mm_M8
- U1: moved to F.Cu
- moved J1 87.7 mm to (680.2, 15.1)
- moved LED6 39.1 mm to (817.6, -7.14)
- moved U1 24.5 mm to (775.5, -15.1), turned to 180 degrees
- moved D104 19.1 mm to (606.4, 13.5), turned to 90 degrees
- moved R3 9.56 mm to (701.7, 57.1)
- moved D100 7.94 mm to (568.3, 13.5), turned to 90 degrees
- moved R1 6.40 mm to (701.7, 47.6)
- moved R11 6.40 mm to (701.7, 60.3)
- moved R2 6.40 mm to (701.7, 50.8)
- moved LED3 5.32 mm to (740.6, 47.6)
- moved R6 5.32 mm to (740.6, 62.7)
- moved LED2 5.02 mm to (735.8, 47.6)
- moved R5 5.02 mm to (735.8, 62.7)
- moved LED1 4.76 mm to (731.0, 47.6)
- moved R4 4.76 mm to (731.0, 62.7)
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Connections:
- U1 pad 8: NMLCK -> Net-(U1-Pad8)
- U1 pad 9: SCLCK -> Net-(U1-Pad9)
Routing:
- net VCC: track 26.7 -> 132.0 mm
- net COL10: track 347.8 -> 272.8 mm
- net SCLCK: track 65.7 -> 0.00 mm
- net COL6: track 553.4 -> 491.5 mm
- net COL5: track 529.9 -> 475.6 mm
- net COL2: track 614.4 -> 563.8 mm, vias 1 -> 0
- net STA1: track 134.8 -> 88.6 mm
- net COL4: track 557.6 -> 513.3 mm
- net STA3: track 127.4 -> 83.5 mm
- net STA2: track 123.3 -> 79.8 mm, vias 1 -> 0
- net COL1: track 602.6 -> 562.1 mm
- net COL7: track 463.3 -> 423.2 mm, vias 1 -> 0
- net COL3: track 554.5 -> 517.9 mm
- net Net-(LED6-Pad2): track 8.06 -> 42.6 mm
- net ROW8: track 430.7 -> 465.1 mm
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Other:
- board size 434.2 x 131.8 mm -> 428.6 x 121.4 mm
- board text added: "A2000 Serotina V1.4 - created by grshaw and bperryman"
- board text removed: "A2000 Serotina V1.3 - created by grshaw and bperryman"
- board text removed: "NMLCK"
- board text removed: "SCLCK"

Commit message: V1.5
1) Remove PCB mount holes from switch footprints.   DONE
Routing:
- net ROW5: track 267.6 -> 299.6 mm
- net ROW10: track 466.1 -> 446.4 mm
- net COL8: track 444.4 -> 463.6 mm, vias 1 -> 0
- net ROW8: track 465.1 -> 452.0 mm
- net COL6: track 491.5 -> 479.4 mm
- net CTRL: track 145.8 -> 134.1 mm, vias 0 -> 1
- net COL9: track 448.2 -> 459.3 mm
- net Net-(MX69-Pad3): track 96.8 -> 85.8 mm
- net ROW6: track 410.6 -> 421.5 mm, vias 0 -> 1
- net Net-(MX33-Pad3): track 252.9 -> 263.0 mm, vias 1 -> 0
- net LALT: track 130.9 -> 121.5 mm, vias 0 -> 1
- net ROW3: track 252.1 -> 260.9 mm
- net COL7: track 423.2 -> 431.9 mm
- net ROW11: track 287.6 -> 295.9 mm
- net COL1: track 562.1 -> 570.4 mm
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Other:
- board text added: "A2000 Serotina V1.5 - created by grshaw and bperryman"
- board text removed: "A2000 Serotina V1.4 - created by grshaw and bperryman"
