File: kicad/a2000Serotina.kicad_pcb (KiCad board)
At the start: 2 copper layers, 428.6 x 121.4 mm, 232 parts, among them J1 90121-0766, U1 Teensy++2.0_(C)

Commit message: Add a2000Serotina_pc_testing_uk.hex
Also complete V1.4 Build instructions and update main README.md with V1.4 pictures.
Parts:
- moved R9 50.5 mm to (819.1, -20.6), turned to 270 degrees
- moved D12 15.7 mm to (666.8, 76.2), turned to 0 degrees
- moved D79 15.7 mm to (642.9, 76.2), turned to 0 degrees
- moved D28 11.9 mm to (661.2, 42.1)
- moved LED2 3.97 mm to (731.8, 47.6)
- moved LED1 3.97 mm to (727.1, 47.6)
- moved LED3 3.97 mm to (736.6, 47.6)
- moved R6 3.97 mm to (736.6, 62.7)
- moved R5 2.38 mm to (733.4, 62.7)
- moved R4 0.79 mm to (730.2, 62.7)
Routing:
- net CPLCK: track 127.1 -> 172.4 mm
- net Net-(LED6-Pad2): track 43.0 -> 3.73 mm
- net GND: track 583.4 -> 620.8 mm
- net COL9: track 459.3 -> 434.7 mm, vias 0 -> 1
- net ROW10: track 446.4 -> 468.9 mm, vias 1 -> 0
- net ROW11: track 295.9 -> 278.1 mm
- net COL2: track 571.4 -> 559.3 mm
- net Net-(D28-Pad2): track 16.7 -> 5.50 mm
- net Net-(MX69-Pad3): track 85.8 -> 96.9 mm
- net Net-(D79-Pad2): track 16.0 -> 5.50 mm
- net Net-(D12-Pad2): track 16.0 -> 5.50 mm
- net CTRL: track 134.1 -> 142.8 mm, vias 1 -> 0
- net ROW9: track 295.1 -> 286.4 mm
- net Net-(MX11-Pad3): track 302.2 -> 309.1 mm, vias 1 -> 0
- net ROW6: track 421.5 -> 414.8 mm
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
Commit message: Add two additional mounting holes
To match WASD PCB.
Parts:
- added H8: MountingHole, MountingHole:MountingHole_2.5mm, F.Cu at (426.9, -18.2)
- added H9: MountingHole, MountingHole:MountingHole_2.5mm, F.Cu at (783.7, 85.7)
Changed lines of the file:
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@@
     (tracks 2043)
     (zones 0)
-    (modules 232)
+    (modules 234)
     (nets 169)
   )
@@
     (add_net VCC)
   )
+  (module MountingHole:MountingHole_2.5mm (layer F.Cu)
+    (at 783.69 85.72)
+    (descr "Mounting Hole 2.5mm, no annular")
+    (tags "mounting hole 2.5mm no annular")
+    (attr virtual)
+    (fp_text reference H9 (at 0 -3.5) (layer F.SilkS)
+      (effects (font (size 1 1) (thickness 0.15)))
+    )
+    (fp_text value MountingHole (at 0 3.5) (layer F.Fab)
+      (effects (font (size 1 1) (thickness 0.15)))
+    )
+    (fp_circle (center 0 0) (end 2.75 0) (layer F.CrtYd) (width 0.05))
+    (fp_circle (center 0 0) (end 2.5 0) (layer Cmts.User) (width 0.15))
+    (fp_text user %R (at 0.3 0) (layer F.Fab)
+      (effects (font (size 1 1) (thickness 0.15)))
+    )
+    (pad 1 np_thru_hole circle (at 0 0) (size 2.5 2.5) (drill 2.5) (layers *.Cu *.Mask))
+  )
+  (module MountingHole:MountingHole_2.5mm (layer F.Cu)
+    (at 426.85 -18.25)
+    (descr "Mounting Hole 2.5mm, no annular")
+    (tags "mounting hole 2.5mm no annular")
+    (attr virtual)
+    (fp_text reference H8 (at 0 -3.5) (layer F.SilkS)
+      (effects (font (size 1 1) (thickness 0.15)))
+    )
+    (fp_text value MountingHole (at 0 3.5) (layer F.Fab)
+      (effects (font (size 1 1) (thickness 0.15)))
+    )
+    (fp_circle (center 0 0) (end 2.75 0) (layer F.CrtYd) (width 0.05))
+    (fp_circle (center 0 0) (end 2.5 0) (layer Cmts.User) (width 0.15))
+    (fp_text user %R (at 0.3 0) (layer F.Fab)
+      (effects (font (size 1 1) (thickness 0.15)))
+    )
+    (pad 1 np_thru_hole circle (at 0 0) (size 2.5 2.5) (drill 2.5) (layers *.Cu *.Mask))
+  )
   (module MX_Alps_Hybrid:MX-6.25U-NoLED (layer F.Cu)
